File: kicad/dc-power-supply.kicad_pcb (KiCad board)
At the start: 2 copper layers, 130 x 265.4 mm, 226 parts, among them IC1 AS4C32M16SA-7TCN, IC2 LT1084, J1 2 Pin Terminal, J2 14 Pin Connector, J3 20 Pin Connector, J4 2 Pin Terminal, J5 30 Pins 0.50 mm Pitch ZIF Con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, J6 14 Pin Connector, J7 20 Pin Connector, J8 10 Pin Connector, J9 USB_B, P1 RB1-125BAG1A, Q1 BC847, Q2 MMBT3906-7-F, Q3 MMBT3906-7-F, Q4 FMMT493TA, SW1 On/Off, SW2 Menu, SW3 Lock/Unlock, SW4 318-ENC130175F-12PS, SW5 Voltage/Amp, U1 LT6657, U10 LT1013DS, U11 LTC2602, U12 LTC3632EDD, U13 LT3081ER, U14 LT3081ER, U15 LPC4337JBD144, U16 LAN8720A, U2 LT8607, U4 LTC3631, U5 LT8612EUDE, U6 LT1013DS, U7 ADuM262N, U8 320S14, U9 LTC2486, Y1 32.768 kHz, Y2 12 MHz, Y3 25MHz

Commit message: Made some major and minor design changes
* Decided on using a 40VAC transformer instead of a toroid. This freed up a lot space for the uC board.
* Switched to a LM338T regulator from TI instead of the more expensive LT part
    - Added protection diode
    - Changed values of feedback resistors to account for minimum load current
* Added a Ferrite bead to +3v3 Rail and used it for reference for the ADC and the DAC. This fixes the Vref > Vcc issue. Don't need the precision 4V supply anymore
* Changed U10B to a Non-inverting Amp with a G = 1000. This gives us a higher voltage to work with. Was originally 0.6mV at max output current.
* Fixed connection issues on U9 where the decoupling caps were connected between +3v3 and the Vcc pin of the chip
* Added datasheets to some parts
* Added mounting holes in the schematic so they stay there in PCB when forward annotation in performed.
* Moved the 12V regulator to a more optimum spot on the board
Parts:
- removed IC2: LT1084, Power_Integrations:TO-220
- removed REF**: Heatsink_Fischer_SK129-STS_42x25mm_2xDrill2.5mm, Heatsinks:Heatsink_Fischer_SK129-STS_42x25mm_2xDrill2.5mm
- removed REF** (x7): MountingHole_2.2mm_M2_DIN965_Pad, Mounting_Holes:MountingHole_2.2mm_M2_DIN965_Pad
- removed REF***: KiCad-Logo2_8mm_SilkScreen, Symbols:KiCad-Logo2_8mm_SilkScreen
- removed REF***: OSHW-Logo_7.5x8mm_SilkScreen, Symbols:OSHW-Logo_7.5x8mm_SilkScreen
- added D14: BAT54, Diode_SMD:D_SOD-323F, F.Cu at (280.0, 221.9)
- added D15: BAT54, Diode_SMD:D_SOD-323F, F.Cu at (263.4, 221.3)
- added H1: MountingHole, MountingHole:MountingHole_2.2mm_M2_Pad, F.Cu at (351.8, 272.8)
- added H10: MountingHole, MountingHole:MountingHole_2.2mm_M2_Pad, F.Cu at (351.5, 143.7)
- added H11: MountingHole, MountingHole:MountingHole_2.2mm_M2_Pad, F.Cu at (351.5, 322.5)
- added H12: MountingHole, MountingHole:MountingHole_2.2mm_M2_Pad, F.Cu at (228.6, 279.8)
- added H2: MountingHole, MountingHole:MountingHole_2.2mm_M2_Pad, F.Cu at (228.2, 322.2)
- added H3: MountingHole, MountingHole:MountingHole_2.2mm_M2_Pad, F.Cu at (227.9, 268.1)
- added H4: MountingHole, MountingHole:MountingHole_2.2mm_M2_Pad, F.Cu at (227.9, 143.7)
- added H5: MountingHole, MountingHole:MountingHole_2.2mm_M2_Pad, F.Cu at (228.2, 63.6)
- added H6: MountingHole, MountingHole:MountingHole_2.2mm_M2_Pad, F.Cu at (228.0, 151.9)
- added H7: MountingHole, MountingHole:MountingHole_2.2mm_M2_Pad, F.Cu at (351.3, 63.7)
- added H8: MountingHole, MountingHole:MountingHole_2.2mm_M2_Pad, F.Cu at (351.7, 279.5)
- added H9: MountingHole, MountingHole:MountingHole_2.2mm_M2_Pad, F.Cu at (351.7, 152.0)
- added L2: Ferrite_Bead_Small, Resistor_SMD:R_1206_3216Metric_Pad1.42x1.75mm_HandSolder, F.Cu at (346.6, 271.3)
- added L7: Ferrite_Bead_Small, Resistor_SMD:R_1206_3216Metric_Pad1.42x1.75mm_HandSolder, F.Cu at (335.0, 271.1)
- added R2: 100k, Resistor_SMD:R_0603_1608Metric, F.Cu at (331.9, 269.2)
- added R5: 1k, Resistor_SMD:R_0603_1608Metric, F.Cu at (331.9, 272.3)
- added U3: LM338T, Package_TO_SOT_THT:TO-220-3_Vertical, F.Cu at (270.9, 220.4)
- R1, R10, R12, R13, R15, R16, R19, R20, R21, R22, R24, R25, R26, R27, R28, R29, R3, R30, R31, R32, R33, R34, R35, R36, R37, R38, R39, R4, R40, R41, R42, R43, R44, R45, R46, R49, R50, R51, R52, R53, R54, R55, R56, R57, R58, R59, R6, R60, R61, R62, R63, R64, R65, R66, R67, R68, R69, R7, R70, R71, R72, R73, R74, R75, R76, R77, R78, R79, R80, R83, R9: footprint Resistors_SMD:R_0603 -> Resistor_SMD:R_0603_1608Metric
- R47, R48: footprint Resistors_SMD:R_1206 -> Resistor_SMD:R_0603_1608Metric
- R81: value 9.2k -> 4.75k; footprint Resistors_SMD:R_0603 -> Resistor_SMD:R_0603_1608Metric
- R82: value 400 -> 200; footprint Resistors_SMD:R_0603 -> Resistor_SMD:R_0603_1608Metric
- R85: footprint Resistors_SMD:R_1210 -> Resistor_SMD:R_0603_1608Metric
- moved R15 98.1 mm to (308.0, 234.0), turned to 270 degrees
- moved D4 97.8 mm to (308.0, 237.2), turned to 90 degrees
- moved R12 97.6 mm to (307.3, 231.3), turned to 0 degrees
- moved R3 94.1 mm to (305.1, 234.1), turned to 270 degrees
- moved R6 93.8 mm to (305.1, 237.1), turned to 270 degrees
- moved C7 92.4 mm to (303.6, 231.3), turned to 180 degrees
- moved U4 86.8 mm to (300.1, 236.1), turned to 0 degrees
- moved C3 79.1 mm to (296.2, 237.5), turned to 270 degrees
- moved L3 78.6 mm to (293.6, 230.8), turned to 180 degrees
- moved Y2 60.8 mm to (312.1, 76.3)
- moved J3 23.5 mm to (314.0, 239.0)
- moved J9 16.1 mm to (254.1, 76.1)
- moved J2 14.6 mm to (319.0, 231.3)
- moved C26 9.05 mm to (350.3, 265.3), turned to 0 degrees
- moved R85 8.66 mm to (256.2, 239.6)
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Connections:
- C42 pad 2: Net-(C42-Pad2) -> GND
- C43 pad 2: Net-(C42-Pad2) -> GND
- IC1 pad 20: Net-(IC1-Pad20) -> (no net)
- IC1 pad 21: Net-(IC1-Pad21) -> (no net)
- IC1 pad 40: Net-(IC1-Pad40) -> (no net)
- J3 pad 5: Net-(J3-Pad5) -> (no net)
- J5 pad 11: Net-(J5-Pad11) -> (no net)
- J5 pad 20: Net-(J5-Pad20) -> (no net)
- J5 pad 21: Net-(J5-Pad21) -> (no net)
- J5 pad 23: Net-(J5-Pad23) -> (no net)
- J7 pad 5: Net-(J7-Pad5) -> (no net)
- J8 pad 7: Net-(J8-Pad7) -> (no net)
- P1 pad R4: Net-(P1-PadR4) -> (no net)
- P1 pad R5: Net-(P1-PadR5) -> (no net)
- P1 pad R6: Net-(P1-PadR6) -> (no net)
- R9 pad 2: +4V -> (no net)
- U1 pad 1: Net-(U1-Pad1) -> (no net)
- U1 pad 5: Net-(U1-Pad5) -> (no net)
- U1 pad 7: Net-(U1-Pad7) -> (no net)
- U1 pad 8: Net-(U1-Pad8) -> (no net)
- U10 pad 6: VOUT -> Net-(R2-Pad1)
- U11 pad 4: +4V -> Net-(L2-Pad1)
- U12 pad 4: Net-(U12-Pad4) -> (no net)
- U12 pad 7: Net-(U12-Pad7) -> (no net)
- U15 pad 1: Net-(U15-Pad1) -> (no net)
- U15 pad 10: Net-(U15-Pad10) -> (no net)
- U15 pad 11: Net-(U15-Pad11) -> (no net)
- U15 pad 112: Net-(U15-Pad112) -> (no net)
- U15 pad 119: Net-(U15-Pad119) -> (no net)
- U15 pad 121: Net-(U15-Pad121) -> (no net)
- U15 pad 127: Net-(U15-Pad127) -> (no net)
- U15 pad 129: Net-(U15-Pad129) -> (no net)
- U15 pad 130: Net-(U15-Pad130) -> (no net)
- U15 pad 136: Net-(U15-Pad136) -> (no net)
- U15 pad 137: Net-(U15-Pad137) -> (no net)
- U15 pad 138: Net-(U15-Pad138) -> (no net)
- U15 pad 139: Net-(U15-Pad139) -> (no net)
- U15 pad 14: Net-(U15-Pad14) -> (no net)
- U15 pad 140: Net-(U15-Pad140) -> (no net)
- U15 pad 142: Net-(U15-Pad142) -> (no net)
- U15 pad 143: Net-(U15-Pad143) -> (no net)
- U15 pad 144: Net-(U15-Pad144) -> (no net)
- U15 pad 15: Net-(U15-Pad15) -> (no net)
- U15 pad 2: Net-(U15-Pad2) -> (no net)
- U15 pad 22: USB0_ID -> (no net)
- U15 pad 29: Net-(U15-Pad29) -> (no net)
- U15 pad 3: Net-(U15-Pad3) -> (no net)
- U15 pad 33: Net-(U15-Pad33) -> (no net)
- U15 pad 35: Net-(U15-Pad35) -> (no net)
- U15 pad 6: Net-(U15-Pad6) -> (no net)
- U15 pad 69: Net-(U15-Pad69) -> (no net)
- U15 pad 7: Net-(U15-Pad7) -> (no net)
- U15 pad 72: Net-(U15-Pad72) -> (no net)
- U15 pad 73: Net-(U15-Pad73) -> (no net)
- U15 pad 79: Net-(U15-Pad79) -> (no net)
- U15 pad 8: Net-(U15-Pad8) -> (no net)
- U15 pad 83: Net-(U15-Pad83) -> (no net)
- U15 pad 85: Net-(U15-Pad85) -> (no net)
- U15 pad 86: Net-(U15-Pad86) -> (no net)
- U15 pad 87: Net-(U15-Pad87) -> (no net)
- U15 pad 88: Net-(U15-Pad88) -> (no net)
- U15 pad 89: Net-(U15-Pad89) -> (no net)
- U15 pad 9: Net-(U15-Pad9) -> (no net)
- U15 pad 90: Net-(U15-Pad90) -> (no net)
- U15 pad 91: Net-(U15-Pad91) -> (no net)
- U15 pad 92: Net-(U15-Pad92) -> (no net)
- U15 pad 93: Net-(U15-Pad93) -> (no net)
- U15 pad 97: Net-(U15-Pad97) -> (no net)
- U15 pad 99: Net-(U15-Pad99) -> (no net)
- U16 pad 10: Net-(U16-Pad10) -> (no net)
- U2 pad 5: Net-(U2-Pad5) -> (no net)
- U2 pad 9: +30V -> GND
- U4 pad 3: Net-(U4-Pad3) -> (no net)
- U4 pad 4: Net-(U4-Pad4) -> (no net)
- U4 pad 7: Net-(U4-Pad7) -> (no net)
- U8 pad 11: Net-(U8-Pad11) -> (no net)
- U8 pad 4: Net-(U8-Pad4) -> (no net)
- U8 pad 5: Net-(U8-Pad5) -> (no net)
- U8 pad 6: Net-(U8-Pad6) -> (no net)
- U8 pad 7: Net-(U8-Pad7) -> (no net)
- U9 pad 11: Net-(U9-Pad11) -> (no net)
- U9 pad 12: Net-(C42-Pad2) -> +3V3
- U9 pad 13: +4V -> Net-(L7-Pad2)
Routing:
- net +30V: track 132.4 -> 205.0 mm, vias 8 -> 0
- net +12V: track 1.97 -> 20.2 mm, vias 0 -> 1
- net +3V3: track 5.61 -> 17.8 mm
- net Net-(C92-Pad1): track 61.3 -> 72.9 mm
- net Net-(J2-Pad2): track 0.00 -> 11.4 mm
- net Net-(J2-Pad9): track 0.00 -> 9.74 mm
- net Net-(J2-Pad6): track 0.00 -> 9.74 mm
- net Net-(J2-Pad4): track 0.00 -> 9.74 mm
- net Net-(J2-Pad10): track 0.00 -> 9.74 mm
- net Net-(J2-Pad7): track 0.00 -> 9.74 mm
- net Net-(J2-Pad13): track 0.00 -> 9.74 mm
- net Net-(J2-Pad11): track 0.00 -> 9.74 mm
- net Net-(J2-Pad12): track 0.00 -> 9.74 mm
- net Net-(J2-Pad8): track 0.00 -> 9.74 mm
- net Net-(J2-Pad14): track 0.00 -> 9.74 mm
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