File: kicad/dc-power-supply.sch (KiCad schematic (older format))
At the start: 0 parts

Commit message: Made some major and minor design changes
* Decided on using a 40VAC transformer instead of a toroid. This freed up a lot space for the uC board.
* Switched to a LM338T regulator from TI instead of the more expensive LT part
    - Added protection diode
    - Changed values of feedback resistors to account for minimum load current
* Added a Ferrite bead to +3v3 Rail and used it for reference for the ADC and the DAC. This fixes the Vref > Vcc issue. Don't need the precision 4V supply anymore
* Changed U10B to a Non-inverting Amp with a G = 1000. This gives us a higher voltage to work with. Was originally 0.6mV at max output current.
* Fixed connection issues on U9 where the decoupling caps were connected between +3v3 and the Vcc pin of the chip
* Added datasheets to some parts
* Added mounting holes in the schematic so they stay there in PCB when forward annotation in performed.
* Moved the 12V regulator to a more optimum spot on the board
Parts:
- added H1, H10, H11, H12, H2, H3, H4, H5, H6, H7, H8, H9: MountingHole, MountingHole:MountingHole_2.2mm_M2_Pad, symbol Mechanical:MountingHole
Other:
- note added: "TODO: Check placement wrt 3D model"
Changed lines of the file:
@@
-EESchema Schematic File Version 2
-LIBS:dc-power-supply
-LIBS:zetex
-LIBS:xilinx
-LIBS:wiznet
-LIBS:video
-LIBS:valves
-LIBS:ttl_ieee
-LIBS:triac_thyristor
-LIBS:transf
-LIBS:switches
-LIBS:supertex
-LIBS:stm8
-LIBS:stm32
-LIBS:siliconi
-LIBS:silabs
-LIBS:relays
-LIBS:references
-LIBS:pspice
-LIBS:powerint
-LIBS:power
-LIBS:philips
-LIBS:opto
-LIBS:onsemi
-LIBS:nxp_armmcu
-LIBS:nxp
-LIBS:nordicsemi
-LIBS:msp430
-LIBS:motors
-LIBS:motorola
-LIBS:motor_drivers
-LIBS:microcontrollers
-LIBS:microchip_pic32mcu
-LIBS:microchip_pic24mcu
-LIBS:microchip_pic18mcu
-LIBS:microchip_pic16mcu
-LIBS:microchip_pic12mcu
-LIBS:microchip_pic10mcu
-LIBS:microchip_dspic33dsc
-LIBS:microchip
-LIBS:memory
-LIBS:mechanical
-LIBS:maxim
-LIBS:linear
-LIBS:leds
-LIBS:ir
-LIBS:interface
-LIBS:intel
-LIBS:infineon
-LIBS:hc11
-LIBS:graphic_symbols
-LIBS:gennum
-LIBS:ftdi
-LIBS:elec-unifil
-LIBS:dsp
-LIBS:diode
-LIBS:digital-audio
-LIBS:device
-LIBS:dc-dc
-LIBS:cypress
-LIBS:contrib
-LIBS:conn
-LIBS:cmos_ieee
-LIBS:cmos4000
-LIBS:brooktre
-LIBS:bosch
-LIBS:bbd
-LIBS:battery_management
-LIBS:audio
-LIBS:atmel
-LIBS:analog_switches
-LIBS:analog_devices
-LIBS:allegro
-LIBS:adc-dac
-LIBS:actel
-LIBS:Zilog
-LIBS:Xicor
-LIBS:Worldsemi
-LIBS:RFSolutions
-LIBS:Power_Management
-LIBS:Oscillators
-LIBS:Lattice
-LIBS:LEM
-LIBS:ESD_Protection
-LIBS:Altera
-LIBS:74xx
-LIBS:74xgxx
-LIBS:transistors
-LIBS:texas
-LIBS:sensors
-LIBS:rfcom
-LIBS:regul
-LIBS:modules
-LIBS:intersil
-LIBS:display
-LIBS:ac-dc
-LIBS:dc-power-supply-cache
-EELAYER 25 0
+EESchema Schematic File Version 4
+EELAYER 30 0
 EELAYER END
 $Descr A4 11693 8268
@@
 Text Notes 2500 5750 0    157  ~ 31
 User Interface Board
+$Comp
+L Mechanical:MountingHole H1
+U 1 1 6071A627
+P 7050 1900
+F 0 "H1" H 7150 1946 50  0000 L CNN
+F 1 "MountingHole" H 7150 1855 50  0000 L CNN
+F 2 "MountingHole:MountingHole_2.2mm_M2_Pad" H 7050 1900 50  0001 C CNN
+F 3 "~" H 7050 1900 50  0001 C CNN
+	1    7050 1900
+	1    0    0    -1
+$EndComp
+$Comp
+L Mechanical:MountingHole H2
+U 1 1 6071B190
+P 7050 2075
+F 0 "H2" H 7150 2121 50  0000 L CNN
+F 1 "MountingHole" H 7150 2030 50  0000 L CNN
+F 2 "MountingHole:MountingHole_2.2mm_M2_Pad" H 7050 2075 50  0001 C CNN
+F 3 "~" H 7050 2075 50  0001 C CNN
+	1    7050 2075
+	1    0    0    -1
+$EndComp
+$Comp
+L Mechanical:MountingHole H3
+U 1 1 6071CC77
+P 7050 2250
+F 0 "H3" H 7150 2296 50  0000 L CNN
+F 1 "MountingHole" H 7150 2205 50  0000 L CNN
+F 2 "MountingHole:MountingHole_2.2mm_M2_Pad" H 7050 2250 50  0001 C CNN
+F 3 "~" H 7050 2250 50  0001 C CNN
+	1    7050 2250
+	1    0    0    -1
+$EndComp
+$Comp
+L Mechanical:MountingHole H4
+U 1 1 6071CC7D
+P 7050 2425
+F 0 "H4" H 7150 2471 50  0000 L CNN
+F 1 "MountingHole" H 7150 2380 50  0000 L CNN
+F 2 "MountingHole:MountingHole_2.2mm_M2_Pad" H 7050 2425 50  0001 C CNN
+F 3 "~" H 7050 2425 50  0001 C CNN
+	1    7050 2425
+	1    0    0    -1
+$EndComp
+$Comp
+L Mechanical:MountingHole H5
+U 1 1 6071D56B
+P 7050 2600
+F 0 "H5" H 7150 2646 50  0000 L CNN
+F 1 "MountingHole" H 7150 2555 50  0000 L CNN
+F 2 "MountingHole:MountingHole_2.2mm_M2_Pad" H 7050 2600 50  0001 C CNN
+F 3 "~" H 7050 2600 50  0001 C CNN
+	1    7050 2600
+	1    0    0    -1
+$EndComp
+$Comp
+L Mechanical:MountingHole H6
+U 1 1 6071D571
+P 7050 2775
+F 0 "H6" H 7150 2821 50  0000 L CNN
+F 1 "MountingHole" H 7150 2730 50  0000 L CNN
+F 2 "MountingHole:MountingHole_2.2mm_M2_Pad" H 7050 2775 50  0001 C CNN
+F 3 "~" H 7050 2775 50  0001 C CNN
+	1    7050 2775
+	1    0    0    -1
+$EndComp
+$Comp
+L Mechanical:MountingHole H7
+U 1 1 6071DC2D
+P 7050 2950
+F 0 "H7" H 7150 2996 50  0000 L CNN
+F 1 "MountingHole" H 7150 2905 50  0000 L CNN
+F 2 "MountingHole:MountingHole_2.2mm_M2_Pad" H 7050 2950 50  0001 C CNN
+F 3 "~" H 7050 2950 50  0001 C CNN
+	1    7050 2950
+	1    0    0    -1
+$EndComp
+$Comp
+L Mechanical:MountingHole H8
+U 1 1 6071DC33
+P 7050 3125
+F 0 "H8" H 7150 3171 50  0000 L CNN
+F 1 "MountingHole" H 7150 3080 50  0000 L CNN
+F 2 "MountingHole:MountingHole_2.2mm_M2_Pad" H 7050 3125 50  0001 C CNN
+F 3 "~" H 7050 3125 50  0001 C CNN
+	1    7050 3125
+	1    0    0    -1
+$EndComp
+$Comp
+L Mechanical:MountingHole H9
+U 1 1 6071F2AB
+P 7050 3300
+F 0 "H9" H 7150 3346 50  0000 L CNN
+F 1 "MountingHole" H 7150 3255 50  0000 L CNN
+F 2 "MountingHole:MountingHole_2.2mm_M2_Pad" H 7050 3300 50  0001 C CNN
+F 3 "~" H 7050 3300 50  0001 C CNN
+	1    7050 3300
+	1    0    0    -1
+$EndComp
+$Comp
+L Mechanical:MountingHole H10
+U 1 1 6071F2B1
+P 7050 3475
+F 0 "H10" H 7150 3521 50  0000 L CNN
+F 1 "MountingHole" H 7150 3430 50  0000 L CNN
+F 2 "MountingHole:MountingHole_2.2mm_M2_Pad" H 7050 3475 50  0001 C CNN
+F 3 "~" H 7050 3475 50  0001 C CNN
+	1    7050 3475
+	1    0    0    -1
+$EndComp
+$Comp
+L Mechanical:MountingHole H11
+U 1 1 6071F2B7
+P 7050 3650
+F 0 "H11" H 7150 3696 50  0000 L CNN
+F 1 "MountingHole" H 7150 3605 50  0000 L CNN
+F 2 "MountingHole:MountingHole_2.2mm_M2_Pad" H 7050 3650 50  0001 C CNN
+F 3 "~" H 7050 3650 50  0001 C CNN
+	1    7050 3650
+	1    0    0    -1
+$EndComp
+$Comp
+L Mechanical:MountingHole H12
+U 1 1 6071F2BD
+P 7050 3825
+F 0 "H12" H 7150 3871 50  0000 L CNN
+F 1 "MountingHole" H 7150 3780 50  0000 L CNN
+F 2 "MountingHole:MountingHole_2.2mm_M2_Pad" H 7050 3825 50  0001 C CNN
+F 3 "~" H 7050 3825 50  0001 C CNN
+	1    7050 3825
+	1    0    0    -1
+$EndComp
+Text Notes 6625 4050 0    60   ~ 0
+TODO: Check placement wrt 3D model
 $EndSCHEMATC
